File: iPadGimbal_Elektronik/iPadGimbal.kicad_pcb (KiCad board)
At the start: 2 copper layers, 92.7 x 58.4 mm, 13 parts, among them J1 Conn_01x05, J2 Conn_01x05, J3 Conn_01x02, J4 Conn_01x02, J5 Conn_01x02, U1 ESP32-DEVKITC-32D, U2 ULN2003A, U3 ULN2003A

Commit message: Silkscreen angepasst
Other:
- board text added: "+5V GND"
- board text removed: "U in"
Changed lines of the file:
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@@
     (property "Sheetname" "")
     (attr through_hole)
-    (fp_text reference "U1" (at -10.829175 -28.446045 -90) (layer "F.SilkS")
+    (fp_text reference "U1" (at -1.27 -28.65 -90) (layer "F.SilkS")
       (effects (font (size 1.000386 1.000386) (thickness 0.15)))
     )
@@
     (effects (font (size 1 1) (thickness 0.15)))
   )
-  (gr_text "U in\n" (at 207.01 97.79 90) (layer "F.SilkS")
+  (gr_text "+5V\n\nGND" (at 207.01 97.79) (layer "F.SilkS")
     (effects (font (size 1 1) (thickness 0.15)))
   )

Commit message: Silkscreen Namen hinzugefügt
Other:
- board text added: "Energieeffiziente Microcontroller WS 2022 Andreas Hagenmeyer & Alexander Riebau"
- board text removed: "Energieeffiziente Microcontroller WS 22"
Changed lines of the file:
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@@
     (property "Sheetname" "")
     (attr smd)
-    (fp_text reference "U3" (at 0 -5.9) (layer "F.SilkS")
+    (fp_text reference "U3" (at -0.04 -2.58) (layer "F.SilkS")
       (effects (font (size 1 1) (thickness 0.15)))
     )
@@
     (property "Sheetname" "")
     (attr through_hole)
-    (fp_text reference "U1" (at -1.27 -28.65 -90) (layer "F.SilkS")
+    (fp_text reference "U1" (at 0 -12.14 -90) (layer "F.SilkS")
       (effects (font (size 1.000386 1.000386) (thickness 0.15)))
     )
@@
     (property "Sheetname" "")
     (attr smd)
-    (fp_text reference "U2" (at 0 -5.9) (layer "F.SilkS")
+    (fp_text reference "U2" (at 0 -2.54) (layer "F.SilkS")
       (effects (font (size 1 1) (thickness 0.15)))
     )
@@
     (effects (font (size 1 1) (thickness 0.15)))
   )
-  (gr_text "Energieeffiziente Microcontroller \nWS 22" (at 181.61 125.73) (layer "F.SilkS")
-    (effects (font (size 1 1) (thickness 0.15)))
+  (gr_text "Energieeffiziente Microcontroller \nWS 2022\nAndreas Hagenmeyer & Alexander Riebau" (at 165.1 125.73) (layer "F.SilkS")
+    (effects (font (size 1 1) (thickness 0.15)) (justify left))
   )
   (gr_text "iPad Gimbal\nV1.0" (at 143.51 77.47) (layer "F.SilkS")

Commit message: Bennenung im Schaltplan korregiert; MassePin des ESP's korregiert
Parts:
- J1, J2: footprint Library:JST_EH_B5B-EH-A_1x05_P2.50mm_Vertical -> Connector_JST:JST_XH_B5B-XH-AM_1x05_P2.50mm_Vertical
- J3, J4: footprint Library:JST_EH_B2B-EH-A_1x02_P2.50mm_Vertical -> Connector_JST:JST_XH_B2B-XH-AM_1x02_P2.50mm_Vertical
- J5, JP1, JP2: footprint Library:PinHeader_1x02_P2.54mm_Vertical -> Connector_PinHeader_2.54mm:PinHeader_1x02_P2.54mm_Vertical
- JP3, JP4: footprint Library:SolderJumper-2_P1.3mm_Open_RoundedPad1.0x1.5mm -> Jumper:SolderJumper-2_P1.3mm_Open_RoundedPad1.0x1.5mm
- U1: footprint Library:MODULE_ESP32-DEVKITC-32D_TWO-ROW -> ESP32-DEVKITC-32D:MODULE_ESP32-DEVKITC-32D_TWO-ROW
- U2, U3: footprint Library:SOIC-16_3.9x9.9mm_P1.27mm -> Package_SO:SOIC-16_3.9x9.9mm_P1.27mm
Connections:
- net M3_S3 renamed M2_S3
- net M4_S4 renamed M2_S4
- U1 pad 14: unconnected-(U1-Pad14) -> GND
Routing:
- net unconnected-(U1-Pad14): track 2.54 -> 0.00 mm
- net GND: track 5.08 -> 7.62 mm
